File: UccMicroDuino/UccMicroDuino.kicad_sch (KiCad schematic)
At the start: 8 parts, among them J2 Conn_01x10_Socket, J2 USB_A, U2 ATtiny85-20S

Commit message: Add files via upload
Parts:
- added D1: 3.6V 1/2mW, Diode_SMD:D_SOD-123, symbol Device:D_Zener
- added D4: Led Green, ledSmd:ledSMD, symbol Device:LED
- added R1 (x2): 68Ω 5% 1/8W, Resistor_SMD:R_0805_2012Metric_Pad1.20x1.40mm_HandSolder, symbol Device:R
- added R1: 330Ω 5% 1/8W, Resistor_SMD:R_0805_2012Metric_Pad1.20x1.40mm_HandSolder, symbol Device:R
- added R4: 330Ω 5% 1/8W, symbol Device:R
- C1: value C -> 0.1 U
- D1: value D_Zener -> 3.6V 1/2mW
- D5: renamed from D3; value LED -> Led Red
- J1: renamed from J2; value USB_A -> USB_PCB_A
- J2: value Conn_01x10_Socket -> Header
- R1: value R -> 1.5K Ω 5% 1/8W
Connections:
- net +5V: now also C1.1, D5.2 (A), J2.1 (Pin_1), U2.8 (VCC)
- net GND: now also C1.2, D1.2 (A), J1.4 (GND), J2.2 (Pin_2), U2.4 (GND), D1.2 (A), R1.2, R4.2
- net at D5.1 (K): now also R4.1
- net at R1.2: now also D1.1 (K), J1.2 (D-), R1.1
- net at U2.1 (~{RESET}/PB5): now also J2.9 (Pin_9)
- net at U2.2 (XTAL1/PB3): now also J2.7 (Pin_7), R1.2
- net at U2.3 (XTAL2/PB4): now also J2.8 (Pin_8), R1.2
- net at U2.5 (AREF/PB0): now also J2.4 (Pin_4)
- net at U2.6 (PB1): now also J2.5 (Pin_5), D4.2 (A)
- net at U2.7 (PB2): now also J2.6 (Pin_6)
- net at J1.1 (VBUS): now also D5.2 (A)
- net at J1.3 (D+): now also D1.1 (K), R1.1
- new net: D4.1 (K), R1.1
- no-connect marks 0 -> 2
Other:
- moved on the sheet: C1, D1, D5, R1, U2
