File: UccMicroDuino/UccMicroDuino.kicad_sch (KiCad schematic)
At the start: 14 parts, among them J1 USB_PCB_A, J2 Header, U2 ATtiny85-20S

Commit message: PCB finalizado
Parts:
- R4: footprint (none) -> Resistor_SMD:R_0805_2012Metric_Pad1.20x1.40mm_HandSolder
- renumbered D1 to D2, D5 to D3, R1 to R2, R1 to R3, R1 to R5, U2 to U1
