File: UccMicroDuino/UccMicroDuino.kicad_sch (KiCad schematic)
At the start: 14 parts, among them J1 USB_PCB_A, J2 Header, U2 ATtiny85-20S

Commit message: cambios de archivos
Parts:
- R4: footprint (none) -> Resistor_SMD:R_0805_2012Metric_Pad1.20x1.40mm_HandSolder
- U2: footprint Package_SO:SOIC-8W_5.3x5.3mm_P1.27mm -> Package_SO:SOIC-8_5.275x5.275mm_P1.27mm
Changed lines of the file:
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@@
       (effects (font (size 1.27 1.27)) (justify right))
     )
-    (property "Footprint" "Package_SO:SOIC-8W_5.3x5.3mm_P1.27mm" (at 177.8 109.22 0)
+    (property "Footprint" "Package_SO:SOIC-8_5.275x5.275mm_P1.27mm" (at 177.8 109.22 0)
       (effects (font (size 1.27 1.27) italic) hide)
     )
@@
       (effects (font (size 1.27 1.27)) (justify left))
     )
-    (property "Footprint" "" (at 256.032 87.63 90)
-      (effects (font (size 1.27 1.27)) hide)
-    )
+    (property "Footprint" "Resistor_SMD:R_0805_2012Metric_Pad1.20x1.40mm_HandSolder" (at 256.032 87.63 90)
+      (effects (font (size 1.27 1.27)) hide)
+    )

Commit message: Arreglando la placa
Parts:
- renumbered D1 to D2, D5 to D3, R1 to R2, R1 to R3, R1 to R5, U2 to U1
