File: UccMicroDuino/UccMicroDuino.kicad_pcb (KiCad board)
At the start: 2 copper layers, 8 parts, among them J1 Conn_01x10_Socket, J2 USB_A, U1 ATtiny85-20S

Commit message: cambios de archivos
Parts:
- added D2: 3.6V 1/2mW, Diode_SMD:D_SOD-123, F.Cu at (118.1, 45.7)
- added D4: Led Green, ledSmd:ledSMD, F.Cu at (124.5, 78.7)
- added R1: 68Ω 5% 1/8W, Resistor_SMD:R_0805_2012Metric_Pad1.20x1.40mm_HandSolder, F.Cu at (124.5, 52.1)
- added R2: 68Ω 5% 1/8W, Resistor_SMD:R_0805_2012Metric_Pad1.20x1.40mm_HandSolder, F.Cu at (129.4, 51.8)
- added R4: 330Ω 5% 1/8W, Resistor_SMD:R_0805_2012Metric_Pad1.20x1.40mm_HandSolder, F.Cu at (109.9, 69.5)
- added R5: 330Ω 5% 1/8W, Resistor_SMD:R_0805_2012Metric_Pad1.20x1.40mm_HandSolder, F.Cu at (118.7, 78.7)
- C1: value C -> 0.1 U
- D1: renamed from D2; value D_Zener -> 3.6V 1/2mW
- D5: renamed from D3; value LED -> Led Red
- J1: renamed from J2; value USB_A -> USB_PCB_A
- J2: renamed from J1; value Conn_01x10_Socket -> Header
- R3: renamed from R1; value R -> 1.5K Ω 5% 1/8W
- U1: footprint Package_SO:SOIC-8W_5.3x5.3mm_P1.27mm -> Package_SO:SOIC-8_5.275x5.275mm_P1.27mm
- moved D1 45.2 mm to (124.5, 45.7), turned to 90 degrees
- moved D3 36.3 mm to (116.8, 53.3), turned to 90 degrees
- moved J1 32.7 mm to (110.1, 48.0)
- moved D5 31.3 mm to (113.7, 66.7)
- moved C1 25.2 mm to (113.7, 70.5), turned to 180 degrees
- moved R3 25.0 mm to (121.3, 52.1), turned to 90 degrees
- moved U1 18.6 mm to (128.7, 63.9), turned to 180 degrees
- moved J2 11.1 mm to (114.9, 74.3), turned to 90 degrees
- renumbered D1 to D3
Connections:
- C1 pad 1: unconnected-(C1-Pad1) -> +5V
- C1 pad 2: unconnected-(C1-Pad2) -> GND
- D1 pad 1: unconnected-(D2-K-Pad1) -> Net-(D1-K)
- D1 pad 2: unconnected-(D2-A-Pad2) -> GND
- D3 pad 2: unconnected-(D1-A-Pad2) -> Net-(D3-A)
- D5 pad 1: unconnected-(D3-K-Pad1) -> Net-(D5-K)
- D5 pad 2: unconnected-(D3-A-Pad2) -> +5V
- J1 pad 1: unconnected-(J2-VBUS-Pad1) -> Net-(D3-A)
- J1 pad 2: unconnected-(J2-D--Pad2) -> Net-(D1-K)
- J1 pad 3: unconnected-(J2-D+-Pad3) -> Net-(D2-K)
- J1 pad 4: unconnected-(J2-GND-Pad4) -> GND
- J2 pad 1: unconnected-(J1-Pin_1-Pad1) -> +5V
- J2 pad 2: unconnected-(J1-Pin_2-Pad2) -> GND
- J2 pad 4: unconnected-(J1-Pin_4-Pad4) -> Net-(J2-Pin_4)
- J2 pad 5: unconnected-(J1-Pin_5-Pad5) -> Net-(D4-A)
- J2 pad 6: unconnected-(J1-Pin_6-Pad6) -> Net-(J2-Pin_6)
- J2 pad 7: unconnected-(J1-Pin_7-Pad7) -> Net-(J2-Pin_7)
- J2 pad 8: unconnected-(J1-Pin_8-Pad8) -> Net-(J2-Pin_8)
- J2 pad 9: unconnected-(J1-Pin_9-Pad9) -> Net-(J2-Pin_9)
- R3 pad 2: unconnected-(R1-Pad2) -> Net-(D1-K)
- U1 pad 1: unconnected-(U1-~{RESET}/PB5-Pad1) -> Net-(J2-Pin_9)
- U1 pad 2: unconnected-(U1-XTAL1/PB3-Pad2) -> Net-(J2-Pin_7)
- U1 pad 3: unconnected-(U1-XTAL2/PB4-Pad3) -> Net-(J2-Pin_8)
- U1 pad 4: unconnected-(U1-GND-Pad4) -> GND
- U1 pad 5: unconnected-(U1-AREF/PB0-Pad5) -> Net-(J2-Pin_4)
- U1 pad 6: unconnected-(U1-PB1-Pad6) -> Net-(D4-A)
- U1 pad 7: unconnected-(U1-PB2-Pad7) -> Net-(J2-Pin_6)
- U1 pad 8: unconnected-(U1-VCC-Pad8) -> +5V
Routing:
- net GND: track 0.00 -> 108.5 mm
- net +5V: track 0.00 -> 43.5 mm
- net Net-(J2-Pin_8): track 0.00 -> 41.9 mm
- net Net-(J2-Pin_7): track 0.00 -> 25.9 mm
- net Net-(D2-K): track 0.00 -> 23.4 mm
- net Net-(D4-A): track 0.00 -> 21.3 mm
- net Net-(D1-K): track 0.00 -> 16.4 mm
- net Net-(J2-Pin_4): track 0.00 -> 16.2 mm
- net Net-(J2-Pin_6): track 0.00 -> 12.9 mm
- net Net-(J2-Pin_9): track 0.00 -> 10.8 mm
- net Net-(D3-A): track 0.00 -> 7.04 mm
- net Net-(D5-K): track 0.00 -> 3.45 mm
- net Net-(D4-K): track 0.00 -> 2.91 mm
Other:
- board outline added: 51.4 x 48.3 mm
