File: UccMicroDuino/UccMicroDuino.kicad_pcb (KiCad board)
At the start: 2 copper layers, 8 parts, among them J1 Conn_01x10_Socket, J2 USB_A, U1 ATtiny85-20S

Commit message: PCB finalizado
Parts:
- added D2: 3.6V 1/2mW, Diode_SMD:D_SOD-123, F.Cu at (133.0, 79.0)
- added D4: Led Green, ledSmd:ledSMD, F.Cu at (153.2, 70.9)
- added R1: 68Ω 5% 1/8W, Resistor_SMD:R_0805_2012Metric_Pad1.20x1.40mm_HandSolder, F.Cu at (143.5, 82.5)
- added R2: 68Ω 5% 1/8W, Resistor_SMD:R_0805_2012Metric_Pad1.20x1.40mm_HandSolder, F.Cu at (143.5, 80.5)
- added R4: 330Ω 5% 1/8W, Resistor_SMD:R_0805_2012Metric_Pad1.20x1.40mm_HandSolder, F.Cu at (155.5, 90.5)
- added R5: 330Ω 5% 1/8W, Resistor_SMD:R_0805_2012Metric_Pad1.20x1.40mm_HandSolder, F.Cu at (140.5, 76.5)
- C1: value C -> 0.1 U
- D1: renamed from D2; value D_Zener -> 3.6V 1/2mW
- D5: renamed from D3; value LED -> Led Red
- J1: renamed from J2; value USB_A -> USB_PCB_A
- J2: renamed from J1; value Conn_01x10_Socket -> Header
- R3: renamed from R1; value R -> 1.5K Ω 5% 1/8W
- moved J2 37.9 mm to (162.0, 69.0)
- moved C1 23.6 mm to (144.5, 90.0), turned to -90 degrees
- moved U1 21.0 mm to (152.5, 79.5), turned to 90 degrees
- moved R3 18.0 mm to (140.5, 88.0), turned to 90 degrees
- moved D5 13.7 mm to (149.6, 89.2), turned to 180 degrees
- moved J1 12.1 mm to (124.2, 81.5)
- moved D1 9.71 mm to (130.0, 81.0), turned to 90 degrees
- moved D3 7.38 mm to (137.0, 87.0), turned to 90 degrees
- renumbered D1 to D3
Connections:
- C1 pad 1: unconnected-(C1-Pad1) -> +5V
- C1 pad 2: unconnected-(C1-Pad2) -> GND
- D1 pad 1: unconnected-(D2-K-Pad1) -> Net-(D1-K)
- D1 pad 2: unconnected-(D2-A-Pad2) -> GND
- D3 pad 2: unconnected-(D1-A-Pad2) -> Net-(D3-A)
- D5 pad 1: unconnected-(D3-K-Pad1) -> Net-(D5-K)
- D5 pad 2: unconnected-(D3-A-Pad2) -> +5V
- J1 pad 1: unconnected-(J2-VBUS-Pad1) -> Net-(D3-A)
- J1 pad 2: unconnected-(J2-D--Pad2) -> Net-(D1-K)
- J1 pad 3: unconnected-(J2-D+-Pad3) -> Net-(D2-K)
- J1 pad 4: unconnected-(J2-GND-Pad4) -> GND
- J2 pad 1: unconnected-(J1-Pin_1-Pad1) -> +5V
- J2 pad 2: unconnected-(J1-Pin_2-Pad2) -> GND
- J2 pad 4: unconnected-(J1-Pin_4-Pad4) -> Net-(J2-Pin_4)
- J2 pad 5: unconnected-(J1-Pin_5-Pad5) -> Net-(D4-A)
- J2 pad 6: unconnected-(J1-Pin_6-Pad6) -> Net-(J2-Pin_6)
- J2 pad 7: unconnected-(J1-Pin_7-Pad7) -> Net-(J2-Pin_7)
- J2 pad 8: unconnected-(J1-Pin_8-Pad8) -> Net-(J2-Pin_8)
- J2 pad 9: unconnected-(J1-Pin_9-Pad9) -> Net-(J2-Pin_9)
- R3 pad 2: unconnected-(R1-Pad2) -> Net-(D1-K)
- U1 pad 1: unconnected-(U1-~{RESET}/PB5-Pad1) -> Net-(J2-Pin_9)
- U1 pad 2: unconnected-(U1-XTAL1/PB3-Pad2) -> Net-(J2-Pin_7)
- U1 pad 3: unconnected-(U1-XTAL2/PB4-Pad3) -> Net-(J2-Pin_8)
- U1 pad 4: unconnected-(U1-GND-Pad4) -> GND
- U1 pad 5: unconnected-(U1-AREF/PB0-Pad5) -> Net-(J2-Pin_4)
- U1 pad 6: unconnected-(U1-PB1-Pad6) -> Net-(D4-A)
- U1 pad 7: unconnected-(U1-PB2-Pad7) -> Net-(J2-Pin_6)
- U1 pad 8: unconnected-(U1-VCC-Pad8) -> +5V
Routing:
- net +5V: track 0.00 -> 47.2 mm
- net Net-(J2-Pin_7): track 0.00 -> 28.1 mm
- net Net-(J2-Pin_8): track 0.00 -> 22.8 mm
- net Net-(D1-K): track 0.00 -> 22.6 mm
- net Net-(J2-Pin_9): track 0.00 -> 20.8 mm
- net Net-(D2-K): track 0.00 -> 18.0 mm
- net Net-(D4-A): track 0.00 -> 15.2 mm
- net Net-(D4-K): track 0.00 -> 14.8 mm
- net Net-(J2-Pin_6): track 0.00 -> 13.4 mm
- net Net-(D3-A): track 0.00 -> 13.1 mm
- net Net-(J2-Pin_4): track 0.00 -> 7.90 mm
- net Net-(D5-K): track 0.00 -> 4.24 mm
- net GND: track 0.00 -> 1.72 mm
- added copper zone on F.Cu, net GND
